File: Store_Board/Kicad/StoreBoard.kicad_sch (KiCad schematic)
At the start: 36 parts, among them J1 Conn_01x10, J2 Conn_01x10, J3 Conn_01x10, J4 Conn_01x10, U1 HM62256BLP, U2 74LS574, U3 74LS32, U4 74LS04, U417 74LS00, U418 74LS00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

Commit message: Further refinements to RAS handling
Parts:
- removed C5, C8: 100nF, Capacitor_THT:C_Disc_D3.0mm_W1.6mm_P2.50mm, symbol Device:C
- removed U3: 74LS32, Package_DIP:DIP-14_W7.62mm, symbol 74xx:74LS32
- removed U4: 74LS04, Package_DIP:DIP-14_W7.62mm, symbol 74xx:74HCT04
- removed U417: 74LS00, Package_DIP:DIP-16_W7.62mm, symbol 74xx:74LS00
- removed unit 6 of U420
Connections:
- net A14M is gone; now on net ~{A14M}: TP1.1 (Pin_1), U1.1 (A14)
- net RAS: now also U418.11, U419.12, U419.13
- net RAS16 renamed ~{RFSHB}
- net RAS32: no longer names the net of TP1.9 (Pin_9)
- no-connect marks 16 -> 11
Other:
- moved on the sheet: C49, C57, R46, R56, U418A, U418B, U418C, U418D, U419A, U419C, U419D, U420A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

Commit message: Final update before test fabrication
Parts:
- added RN1, RN2: 33Ω, Package_DIP:DIP-16_W7.62mm, symbol Device:R_Pack08
Connections:
- net ~{RFSHB} is gone; now on net ~{RFRSHB}: TP1.7 (Pin_7)
- net A0: now also RN1.16 (R1.2)
- net A1: now also RN1.15 (R2.2)
- net A2: now also RN1.14 (R3.2)
- net A3: now also RN1.13 (R4.2)
- net A4: now also RN1.12 (R5.2)
- net A5: now also RN1.11 (R6.2)
- net A6: now also RN1.10 (R7.2)
- net M1,1: now also RN2.4 (R4.1); no longer RN54.5 (R4), U1.15 (Q3)
- net M1,3: now also RN1.1 (R1.1)
- net M1,4: now also RN1.2 (R2.1)
- net M1,5: now also RN1.4 (R4.1)
- net M1,6: now also RN1.6 (R6.1)
- net M2,10: now also RN2.6 (R6.1); no longer RN54.7 (R6), U1.17 (Q5)
- net M3,4: now also RN1.3 (R3.1)
- net M3,5: now also RN1.5 (R5.1)
- net M3,6: now also RN1.7 (R7.1)
- net M4,10: now also RN2.5 (R5.1); no longer RN54.6 (R5), U1.16 (Q4)
- net M4,3: now also RN2.8 (R8.1); no longer RN54.9 (R8), U1.19 (Q7)
- net M4,6: now also RN2.1 (R1.1); no longer RN54.2 (R1), U1.11 (Q0)
- net M4,7: now also RN2.2 (R2.1); no longer RN54.3 (R2), U1.12 (Q1)
- net M4,8: now also RN2.3 (R3.1); no longer RN54.4 (R3), U1.13 (Q2)
- net M4,9: now also RN2.7 (R7.1); no longer RN54.8 (R7), U1.18 (Q6)
- net ROW: now also TP1.9 (Pin_9)
- net ~{CAS}: now also RN1.9 (R8.2); no longer U421.7 (~{Q})
- new net D0: RN2.16 (R1.2), RN54.2 (R1), U1.11 (Q0)
- new net D1: RN2.15 (R2.2), RN54.3 (R2), U1.12 (Q1)
- new net D2: RN2.14 (R3.2), RN54.4 (R3), U1.13 (Q2)
- new net D3: RN2.13 (R4.2), RN54.5 (R4), U1.15 (Q3)
- new net D4: RN2.12 (R5.2), RN54.6 (R5), U1.16 (Q4)
- new net D5: RN2.11 (R6.2), RN54.7 (R6), U1.17 (Q5)
- new net D6: RN2.10 (R7.2), RN54.8 (R7), U1.18 (Q6)
- new net D7: RN2.9 (R8.2), RN54.9 (R8), U1.19 (Q7)
- new net ~{CAS}_PRE: RN1.8 (R8.1), U421.7 (~{Q})
- no-connect marks 11 -> 10

Commit message: Corrected footprints
Parts:
- removed RN1, RN2: 33Ω, Package_DIP:DIP-16_W7.62mm, symbol Device:R_Pack08
- J1, J2, J3, J4: footprint Connector_JST:JST_EH_B10B-EH-A_1x10_P2.50mm_Vertical -> Connector_PinHeader_2.54mm:PinHeader_1x10_P2.54mm_Vertical
- R46, R56: footprint Resistor_THT:R_Axial_DIN0204_L3.6mm_D1.6mm_P5.08mm_Horizontal -> Resistor_THT:R_Axial_DIN0207_L6.3mm_D2.5mm_P10.16mm_Horizontal
- U418, U419, U420, U422: footprint Package_DIP:DIP-16_W7.62mm -> Package_DIP:DIP-14_W7.62mm
Connections:
- net D0 is gone; now on net M4,6: RN54.2 (R1), U1.11 (Q0)
- net D1 is gone; now on net M4,7: RN54.3 (R2), U1.12 (Q1)
- net D2 is gone; now on net M4,8: RN54.4 (R3), U1.13 (Q2)
- net D3 is gone; now on net M1,1: RN54.5 (R4), U1.15 (Q3)
- net D4 is gone; now on net M4,10: RN54.6 (R5), U1.16 (Q4)
- net D5 is gone; now on net M2,10: RN54.7 (R6), U1.17 (Q5)
- net D6 is gone; now on net M4,9: RN54.8 (R7), U1.18 (Q6)
- net D7 is gone; now on net M4,3: RN54.9 (R8), U1.19 (Q7)
- net ~{CAS}_PRE is gone; now on net ~{CAS}: U421.7 (~{Q})
- net ROW: no longer TP1.9 (Pin_9)
- net ~{WE}: now reaches U1.27 (~{WE}), U423.6
- net ~{WE}: now also TP1.9 (Pin_9)
